File: ARDF-80m-RX-with-SA612/ARDF-80m-rx.kicad_sch (KiCad schematic)
At the start: 40 parts, among them J4 AudioJack3_SwitchTR, Q1 BC847, Q4 BC847, SW2 SW_SPDT, U1 L78L06_TO92, U3 LM358, Y2 3.5795 MHz

Commit message: Add schematic and PCB pdf exports and interactive BOM
Other:
- company: (none) -> HA3PB
- title: (none) -> ARDF 80m RX - SA612 version
Changed lines of the file:
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@@
 	(generator_version "9.0")
 	(paper "A4")
+	(title_block
+		(title "ARDF 80m RX - SA612 version")
+		(date "2025-06-28")
+		(company "HA3PB")
+		(comment 1 "Weisz Pál")
+	)
 	(junction
 		(at 43.18 91.44)
