File: Puya-80m-Fox/Puya-80m-Fox-HW/Puya-80m-Fox.kicad_sch (KiCad schematic)
At the start: 27 parts, among them J1 ANT, J2 PROG, J3 UART, J4 KEY, Q1 FHK3401, Q2 BC847, Q4 BC847, U6 LD1117S33TR_SOT223, Y1 3579kHz

Commit message: Add schematic and PCB pdf exports and interactive BOM
Other:
- company: (none) -> HA3PB
- title: (none) -> Puya-80m-Fox
Changed lines of the file:
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@@
 	(generator_version "9.0")
 	(paper "A4")
+	(title_block
+		(title "Puya-80m-Fox")
+		(date "2025-06-28")
+		(company "HA3PB")
+		(comment 1 "Weisz Pál")
+	)
 	(text "PA10 AF8 USART1_TX\nPA3 AF1 USART1_RX\nPA1 AF13 TIM1_CH4"
 		(exclude_from_sim no)
